File: Tone_Master/Tone_Master.kicad_sch (KiCad schematic)
At the start: 68 parts, among them J2 Barrel_Jack, Q1 2N3904, Q2 2N3904, SW1 SW_Rotary_3x4, U1 TL072, U2 TL072, U3 TL072, U8 LM386

Commit message: Replace pdf with project circuit version
Parts:
- removed C1, C2: 47uF, Capacitor_THT:CP_Radial_D8.0mm_P5.00mm, symbol Device:C_Polarized_Small_US
- removed C10, C4: 1uF, Capacitor_THT:C_Rect_L7.2mm_W3.0mm_P5.00mm_FKS2_FKP2_MKS2_MKP2, symbol Device:C
- removed C11, C3: 470nF, Capacitor_THT:C_Rect_L7.2mm_W3.0mm_P5.00mm_FKS2_FKP2_MKS2_MKP2, symbol Device:C
- removed C13: 100n, Capacitor_THT:C_Rect_L7.2mm_W3.0mm_P5.00mm_FKS2_FKP2_MKS2_MKP2, symbol Device:C
- removed C15, C7: 100pF, Capacitor_THT:C_Rect_L7.2mm_W3.0mm_P5.00mm_FKS2_FKP2_MKS2_MKP2, symbol Device:C
- removed C5: 22nF, Capacitor_THT:C_Rect_L7.2mm_W3.0mm_P5.00mm_FKS2_FKP2_MKS2_MKP2, symbol Device:C
- removed C9: 100p, Capacitor_THT:C_Radial_D5.0mm_H7.0mm_P2.00mm, symbol Device:C
- removed D1, D2, D3: 1N4148, Diode_THT:D_DO-35_SOD27_P7.62mm_Horizontal, symbol Diode:1N4148
- removed D4, D5: LED, LED_THT:LED_D3.0mm_Clear, symbol Device:LED
- removed R1, R2: 47k, Resistor_THT:R_Axial_DIN0309_L9.0mm_D3.2mm_P12.70mm_Horizontal, symbol Device:R
- removed R11: 1k, Resistor_THT:R_Axial_DIN0309_L9.0mm_D3.2mm_P12.70mm_Horizontal, symbol Device:R
- removed R12: 10k, Resistor_THT:R_Axial_DIN0309_L9.0mm_D3.2mm_P12.70mm_Horizontal, symbol Device:R
- removed R14: 680K, Resistor_THT:R_Axial_DIN0309_L9.0mm_D3.2mm_P12.70mm_Horizontal, symbol Device:R
- removed R3, R4: 1Meg, Resistor_THT:R_Axial_DIN0309_L9.0mm_D3.2mm_P12.70mm_Horizontal, symbol Device:R
- removed R5, R6: 10K, Resistor_THT:R_Axial_DIN0309_L9.0mm_D3.2mm_P12.70mm_Horizontal, symbol Device:R
- removed RV1: 100k, Potentiometer_THT:Potentiometer_Piher_PT-15-V02_Vertical, symbol Device:R_Potentiometer
- removed unit 3 of U1
- removed U2, U3: TL072, Package_DIP:DIP-8_W7.62mm, symbol Amplifier_Operational:TL072
- added C29: 1uF, Capacitor_THT:CP_Radial_D8.0mm_P5.00mm, symbol Device:C_Polarized_Small_US
- added C30, C35, C39: 470nF, Capacitor_THT:C_Rect_L7.2mm_W3.0mm_P5.00mm_FKS2_FKP2_MKS2_MKP2, symbol Device:C
- added C31, C34: 47uF, Capacitor_THT:CP_Radial_D8.0mm_P5.00mm, symbol Device:C_Polarized_Small_US
- added C32, C37: 220n, Capacitor_THT:C_Rect_L7.2mm_W3.0mm_P5.00mm_FKS2_FKP2_MKS2_MKP2, symbol Device:C
- added C33: 50pF, Capacitor_THT:C_Radial_D5.0mm_H7.0mm_P2.00mm, symbol Device:C
- added C36: 22nF, Capacitor_THT:C_Rect_L7.2mm_W3.0mm_P5.00mm_FKS2_FKP2_MKS2_MKP2, symbol Device:C
- added C38: 50pF, Capacitor_THT:C_Rect_L7.2mm_W3.0mm_P5.00mm_FKS2_FKP2_MKS2_MKP2, symbol Device:C
- added C40: 100pF, Capacitor_THT:C_Rect_L7.2mm_W3.0mm_P5.00mm_FKS2_FKP2_MKS2_MKP2, symbol Device:C
- added C41: 1uF, Capacitor_THT:C_Rect_L7.2mm_W3.0mm_P5.00mm_FKS2_FKP2_MKS2_MKP2, symbol Device:C
- added C42: 10n, Capacitor_THT:C_Rect_L7.2mm_W3.0mm_P5.00mm_FKS2_FKP2_MKS2_MKP2, symbol Device:C
- added D10: LED, symbol Device:LED
- added D6, D7, D8: 1N4148, Diode_THT:D_DO-35_SOD27_P7.62mm_Horizontal, symbol Diode:1N4148
- added D9: LED, LED_SMD:LED_1206_3216Metric_Pad1.42x1.75mm_HandSolder, symbol Device:LED
- added R18: 10K, Resistor_THT:R_Axial_DIN0309_L9.0mm_D3.2mm_P12.70mm_Horizontal, symbol Device:R
- added R28: 500, Resistor_THT:R_Axial_DIN0309_L9.0mm_D3.2mm_P12.70mm_Horizontal, symbol Device:R
- added R29, R32: 47k, Resistor_SMD:R_0805_2012Metric_Pad1.20x1.40mm_HandSolder, symbol Device:R
- added R30: 1Meg, Resistor_SMD:R_0805_2012Metric_Pad1.20x1.40mm_HandSolder, symbol Device:R
- added R31: 1K, Resistor_SMD:R_0805_2012Metric_Pad1.20x1.40mm_HandSolder, symbol Device:R
- added R33, R36: 1k, Resistor_SMD:R_0805_2012Metric_Pad1.20x1.40mm_HandSolder, symbol Device:R
- added R34: 10k, Resistor_SMD:R_0805_2012Metric_Pad1.20x1.40mm_HandSolder, symbol Device:R
- added R35: 680K, Resistor_SMD:R_0805_2012Metric_Pad1.20x1.40mm_HandSolder, symbol Device:R
- added R37: 22K, Resistor_SMD:R_0805_2012Metric_Pad1.20x1.40mm_HandSolder, symbol Device:R
- added R38: 100K, Resistor_SMD:R_0805_2012Metric_Pad1.20x1.40mm_HandSolder, symbol Device:R
- added RV5: 100K, Potentiometer_THT:Potentiometer_Piher_PT-15-V02_Vertical, symbol Device:R_Potentiometer
- added U3: TL072, Package_DIP:DIP-8_W7.62mm, symbol Amplifier_Operational:TL072
- added U4: TL072, symbol Amplifier_Operational:TL072
- C14: value 220n -> 50pF
- C17: value 10nF -> 100nF
- C6: value 10nF -> 10n
- J2: value Barrel_Jack -> Audio_Jack
- R13: value 1K -> 10K; footprint Resistor_THT:R_Axial_DIN0309_L9.0mm_D3.2mm_P12.70mm_Horizontal -> Resistor_SMD:R_0805_2012Metric_Pad1.20x1.40mm_HandSolder
- R16: value 22K -> 2.2K
- R19: value 22k -> 1Meg; footprint Resistor_THT:R_Axial_DIN0309_L9.0mm_D3.2mm_P12.70mm_Horizontal -> Resistor_SMD:R_0805_2012Metric_Pad1.20x1.40mm_HandSolder
- R27: value 1Meg -> 10K; footprint Resistor_THT:R_Axial_DIN0309_L9.0mm_D3.2mm_P12.70mm_Horizontal -> Resistor_SMD:R_0805_2012Metric_Pad1.20x1.40mm_HandSolder
- U1: footprint Package_DIP:DIP-8_W7.62mm -> (none)
Connections:
- net +9V: now also C34.1, R32.2
- net 4.5V_ref: now also R19.2, C31.1, R29.2, R30.2, R32.1, U4.5 (+)
- net DISTORT_OUT: now also SW1.2, C42.1, D10.1 (K), D9.2 (A), R36.1; no longer C16.2, C6.2, R16.2, R27.1
- net FUZZ_IN: now also SW1.14; no longer SW1.11
- net GND: now also C14.2, C31.2, C32.1, C34.2, C37.2, C42.2, D10.2 (A), D9.1 (K), R28.1, R29.1; no longer C14.1, C23.2, C26.1, C27.2, R27.2, SW1.7, U8.4 (GND)
- net PICKUP_OUT: now also R13.2, R27.2, SW1.7, R18.1; no longer SW1.15
- net at U1.3 (+): now also R19.1, C36.2
- net at U1.1: now also C38.1, C39.2, R38.1; no longer R19.2
- net OD_OUT: now reaches SW1.1
- net OD_OUT: now also C35.2; no longer R19.1
- net at R13.1: now also C14.1, C36.1; no longer C14.2
- net at Q1.1 (E), R10.1: now also C12.1, R28.2; no longer R13.2, U1.2 (-)
- net OUT: now reaches SW1.13
- net OUT: now also C16.2, R16.2
- net FUZZ_OUT: now reaches SW1.3
- net FUZZ_OUT: now also C6.2; no longer C12.1
- net Direct_OUT: now reaches SW1.4
- net Direct_OUT: now also C29.2
- removed net Preamp_IN: C20.1, SW1.10, SW1.12, SW1.9
- net Preamp_OUT: no longer names the net of R26.2, U1.7
- net Preamp_OUT: now also C29.1
- new net: C33.2, C35.1, D7.2 (A), D8.1 (K), R37.2, U3.1
- new net: C37.1, R33.1
- new net: C38.2, R33.2, R38.2, U1.2 (-)
- new net: C41.1, R36.2
- new net: C40.1, C41.2, R35.1, U4.7
- new net: C30.2, R30.1, U3.3 (+)
- new net: C40.2, R34.1, R35.2, U4.6 (-)
- new net: C32.2, R31.1
- new net: C33.1, D6.2 (A), D7.1 (K), R31.2, RV5.3, U3.2 (-)
- new net: C30.1, R27.1
- new net: C20.1, R18.2
- new net: R37.1, RV5.2
- new net: D6.1 (K), D8.2 (A)
- new net: C39.1, R34.2
- new net GNDPWR: C23.2, C26.1, C27.2, U8.4 (GND)
- no-connect marks 4 -> 2
Other:
- note added: "Drive"
- note removed: "Drive/Gain/Fuzz"
- note removed: "POWER"
- moved on the sheet: C12, C16, C17, C18, C19, C20, C21, C23, C24, C25, C26, C27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
